File: esc.kicad_pcb (KiCad board)
At the start: 2 copper layers, 99 x 50 mm, 210 parts, among them J1 Conn_01x05_Socket, J2 Conn_01x03_Socket, Q1 FDMS86550, Q10 FDMS86550, Q11 FDMS86550, Q12 FDMS86550, Q2 FDMS86550, Q3 FDMS86550, Q4 FDMS86550, Q5 FDMS86550, Q6 FDMS86550, Q7 FDMS86550, Q8 FDMS86550, Q9 FDMS86550, U1 STM32F103C8Tx, U10 TLV9061xDBV, U11 TLV9061xDBV, U12 TLV9061xDBV, U2 AOZ1284PI, U3 TLV9061xDBV, U4 UCC27282DRCT, U5 UCC27282DRCT, U6 UCC27282DRCT, U7 TLV9061xDBV, U8 TLV9061xDBV, Y1 8Mhz

Commit message: init
Parts:
- removed R31, R40, R76, R83: 10k_1206, Resistor_SMD:R_1206_3216Metric
- removed R71, R75: 10k_603, Resistor_SMD:R_0603_1608Metric
- removed the R90 at (243.6, 72.7)
- C23, C24, C26, C39, C40, C41, C44, C6, C7, R49, R55, R56, R57, R60, R62, R64, R65, R66, R67, R72, U7, U8: moved to B.Cu
- C31: moved to F.Cu
- D1: value 1N62xxCA -> CDBA540-HF; footprint Diode_THT:D_DO-201AE_P15.24mm_Horizontal -> Diode_SMD:D_SMA
- F1: footprint Fuse:Fuse_0402_1005Metric -> Library:FUSE_3557-2
- moved D1 198.1 mm to (56.8, 50.2), turned to 180 degrees
- moved R81 181.0 mm to (69.0, 110.5)
- moved R85 174.7 mm to (71.2, 98.2)
- moved D20 171.4 mm to (73.0, 57.9), turned to -90 degrees
- moved D21 168.5 mm to (81.8, 45.7)
- moved D16 166.7 mm to (78.8, 57.9), turned to -90 degrees
- moved D19 165.6 mm to (84.8, 45.7), turned to 180 degrees
- moved R58 162.1 mm to (75.8, 57.3), turned to -90 degrees
- moved D17 157.5 mm to (87.5, 57.7), turned to -90 degrees
- moved R50 151.4 mm to (81.7, 57.3), turned to -90 degrees
- moved R51 148.8 mm to (84.7, 57.4), turned to -90 degrees
- moved D18 146.6 mm to (98.0, 57.4), turned to -90 degrees
- moved D25 145.6 mm to (106.8, 45.4)
- moved D14 142.8 mm to (93.3, 57.7), turned to -90 degrees
- moved R80 142.7 mm to (100.9, 57.0), turned to -90 degrees
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Connections:
- C17 pad 1: VCC -> +3v3
- C23 pad 2: GND -> MCU_GND
- C24 pad 2: GND -> MCU_GND
- C26 pad 2: GND -> MCU_GND
- C27 pad 2: GND -> MCU_GND
- C28 pad 2: GND -> MCU_GND
- C35 pad 1: VCC -> +3v3
- C36 pad 1: VCC -> +3v3
- C39 pad 1: VCC -> +3v3
- C40 pad 1: VCC -> +3v3
- C43 pad 2: GND -> MCU_GND
- C51 pad 1: VCC -> +3v3
- C6 pad 2: GND -> MCU_GND
- C7 pad 2: GND -> MCU_GND
- D1 pad 1: GND -> VIN
- D1 pad 2: VIN -> GND
- J2 pad 1: User_UART_Rx -> User_UART_Tx
- R68 pad 2: GND -> MCU_GND
- R7 pad 2: GND -> MCU_GND
- R90 pad 2: GND -> MCU_GND
- S8 pad 1: GND -> MCU_GND
- U1 pad 23: GND -> MCU_GND
- U1 pad 35: GND -> MCU_GND
- U1 pad 42: User_UART_Rx -> User_UART_Tx
- U1 pad 47: GND -> MCU_GND
- U1 pad 8: GND -> MCU_GND
- U10 pad 5: VCC -> +3v3
- U11 pad 5: VCC -> +3v3
- U12 pad 5: VCC -> +3v3
- U3 pad 5: VCC -> +3v3
- U7 pad 5: VCC -> +3v3
- U8 pad 5: VCC -> +3v3
Routing:
- net +3V3: track 78.4 -> 0.00 mm
- net GND: track 65.8 -> 0.00 mm, vias 4 -> 0
- net MCU_RST: track 49.4 -> 0.00 mm
- net MCU_SWDIO: track 32.6 -> 0.00 mm
- net User_UART_Rx: track 31.8 -> 0.00 mm
- net MCU_SWCLK: track 31.0 -> 0.00 mm
- net Net-(D13-A): track 28.4 -> 0.04 mm, vias 2 -> 0
- net Phase_C_HO: track 22.6 -> 0.00 mm
- net Net-(D11-K): track 21.8 -> 0.00 mm
- net Net-(D7-A): track 19.8 -> 0.45 mm
- net Net-(D29-A): track 16.1 -> 0.01 mm
- net User_LED_3: track 14.1 -> 0.00 mm
- net VCC: track 13.9 -> 0.00 mm
- net User_LED_2: track 12.2 -> 0.00 mm
- net User_LED_1: track 9.89 -> 0.00 mm
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Other:
- board size 99 x 50 mm -> 223.7 x 149.7 mm
- board text removed: "Bu gnd isole ngd olcan 3v3 gnd sinden farklı"

Commit message: bitti sayılır
Parts:
- removed D10: CDBA540-HF, Diode_SMD:D_SMA
- removed High_Mos_A1, High_Mos_B1, High_Mos_C1, Low_Mos_A1, Low_Mos_B1, Low_Mos_C1, TP7, TP8: TestPoint, TestPoint:TestPoint_Pad_1.5x1.5mm
- removed R32, R41, R48, R53: 10k_603, Resistor_SMD:R_0603_1608Metric
- removed R54, R61: 10k_1206, Resistor_SMD:R_1206_3216Metric
- removed the R68 at (238.0, 69.4)
- added C45: 330uF, Capacitor_SMD:C_Elec_10x10.2, B.Cu at (176.0, 105.6)
- added J5: Conn_01x01_Pin, Connector_Pin:Pin_D1.3mm_L11.0mm_LooseFit, F.Cu at (175.5, 116.8)
- added J6: Conn_01x01_Pin, Connector_Pin:Pin_D1.3mm_L11.0mm_LooseFit, F.Cu at (150.2, 116.8)
- added J7: Conn_01x01_Pin, Connector_Pin:Pin_D1.3mm_L11.0mm_LooseFit, F.Cu at (122.9, 116.8)
- added J8: Conn_01x01_Pin, Connector_Pin:Pin_D1.3mm_L11.0mm_LooseFit, F.Cu at (95.3, 99.3)
- added J9: Conn_01x01_Pin, Connector_Pin:Pin_D1.3mm_L11.0mm_LooseFit, F.Cu at (95.3, 108.0)
- C11, C16, C17, C21, C22, C35, C36, C38, C42, C51, C52, C53, C54, R18, R19, R20, R33, R34, R35, R36, R37, R59, R6, R77, R78, R79, R81, R82, R84, R85, R86, R87, R88, R89, R9, U10, U11, U12, U3: moved to B.Cu
- C25: value 100n -> 330uF; footprint Capacitor_SMD:C_0603_1608Metric -> Capacitor_SMD:C_Elec_10x10.2; moved to B.Cu
- C8: value 100n_603 -> 330uF; footprint Capacitor_SMD:C_0603_1608Metric -> Capacitor_SMD:C_Elec_10x10.2; moved to B.Cu
- moved R59 110.7 mm to (132.2, 30.1), turned to 180 degrees
- moved C16 109.6 mm to (144.7, 33.7), turned to 180 degrees
- moved R81 109.5 mm to (144.7, 31.3), turned to 180 degrees
- moved C8 108.5 mm to (124.1, 105.7), turned to 90 degrees
- moved R82 104.6 mm to (156.3, 97.6), turned to -90 degrees
- moved R88 103.0 mm to (161.0, 109.2), turned to 180 degrees
- moved C53 102.8 mm to (144.7, 28.9), turned to 180 degrees
- moved R85 102.7 mm to (144.7, 26.4), turned to 180 degrees
- moved R9 102.4 mm to (132.4, 26.4), turned to 180 degrees
- moved C54 101.9 mm to (161.0, 107.7), turned to 180 degrees
- moved R84 101.7 mm to (153.6, 94.0)
- moved C25 101.2 mm to (150.1, 105.6), turned to 90 degrees
- moved R89 98.5 mm to (161.0, 106.1)
- moved R86 97.1 mm to (164.2, 99.2), turned to 90 degrees
- moved R87 92.7 mm to (164.2, 96.2), turned to 90 degrees
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Connections:
- C25 pad 1: +3V3 -> VCC
- C8 pad 1: VIN -> VCC
Routing:
- net (no net): track 0.60 -> 0.00 mm
Other:
- board size 223.7 x 149.7 mm -> 177.6 x 143.1 mm
