File: esc.kicad_sch (KiCad schematic)
At the start: 205 parts, among them J1 Conn_01x05_Socket, J2 Conn_01x03_Socket, Q1 FDMS86550, Q10 FDMS86550, Q11 FDMS86550, Q12 FDMS86550, Q2 FDMS86550, Q3 FDMS86550, Q4 FDMS86550, Q5 FDMS86550, Q6 FDMS86550, Q7 FDMS86550, Q8 FDMS86550, Q9 FDMS86550, U1 STM32F103C8Tx, U10 TLV9061xDBV, U11 TLV9061xDBV, U12 TLV9061xDBV, U2 AOZ1284PI, U3 TLV9061xDBV, U4 UCC27282DRCT, U5 UCC27282DRCT, U6 UCC27282DRCT, U7 TLV9061xDBV, U8 TLV9061xDBV, Y1 8Mhz

Commit message: init
Parts:
- removed D1: 1N62xxCA, Diode_THT:D_DO-201AE_P15.24mm_Horizontal, symbol Diode:1N62xxCA
- removed R31, R40, R54, R61, R76, R83: 10k_1206, Resistor_SMD:R_1206_3216Metric, symbol Device:R_Small
- removed R32, R41, R48, R53, R71, R75: 10k_603, Resistor_SMD:R_0603_1608Metric, symbol Device:R_Small
- added D1: CDBA540-HF, Diode_SMD:D_SMA, symbol Diode:CDBA340-HF
- F1: footprint Fuse:Fuse_0402_1005Metric -> Library:FUSE_3557-2
Connections:
- net +3v3: now also C17.1, C35.1, C36.1, C39.1, C40.1, C51.1, U10.5 (V+), U11.5 (V+), U12.5 (V+), U3.5 (V+), U7.5 (V+), U8.5 (V+)
- net GND: now also D1.2 (A); no longer C23.2, C24.2, C26.2, C27.2, C28.2, C43.2, C6.2, C7.2, R68.2, R7.2, R90.2, S8.1, U1.23 (VSS), U1.35 (VSS), U1.47 (VSS), U1.8 (VSSA)
- net User_UART_Rx: no longer J2.1 (Pin_1), U1.42 (PB6)
- net VCC: no longer C17.1, C35.1, C36.1, C39.1, C40.1, C51.1, U10.5 (V+), U11.5 (V+), U12.5 (V+), U3.5 (V+), U7.5 (V+), U8.5 (V+)
- net VIN: now also D1.1 (K)
- new net MCU_GND: C23.2, C24.2, C26.2, C27.2, C28.2, C43.2, C6.2, C7.2, R68.2, R7.2, R90.2, S8.1, U1.23 (VSS), U1.35 (VSS), U1.47 (VSS), U1.8 (VSSA)
- new net User_UART_Tx: J2.1 (Pin_1), U1.42 (PB6)
Other:
- moved on the sheet: F1, R49

Commit message: bitti sayılır
Parts:
- removed High_Mos_A1, High_Mos_B1, High_Mos_C1, Low_Mos_A1, Low_Mos_B1, Low_Mos_C1, TP7, TP8: TestPoint, TestPoint:TestPoint_Pad_1.5x1.5mm, symbol Connector:TestPoint
- added C25, C45, C8: 330uF, Capacitor_SMD:C_Elec_10x10.2, symbol Device:C_Polarized_Small
- added J5, J6, J7, J8, J9: Conn_01x01_Pin, Connector_Pin:Pin_D1.3mm_L11.0mm_LooseFit, symbol Connector:Conn_01x01_Pin
Connections:
- net GND: now also C25.2, C45.2, C8.2, J8.1 (Pin_1)
- net VCC: now also C25.1, C45.1, C8.1, J9.1 (Pin_1)
- net VPH_A: now also J7.1 (Pin_1)
- net VPH_B: now also J6.1 (Pin_1)
- net VPH_C: now also J5.1 (Pin_1)
- no-connect marks 19 -> 11
Other:
- moved on the sheet: F1
